File: Schematica/Autogradina.kicad_sch (KiCad schematic)
At the start: 50 parts, among them J1 Power_Connector, J2 AC_Connector, J3 UART_Connector, J4 USB_B_Micro, J5 Boot_Jumper, J6 Ports_Connector, J7 Conn_01x02_Socket, J8 Conn_01x02_Socket, J9 Conn_01x02_Socket, K1 G5LE-1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

Commit message: Finished up
Parts:
- added NT1: NetTie_2, NetTie:NetTie-2_SMD_Pad0.5mm, symbol Device:NetTie_2
Connections:
- net AC_G: now also NT1.1; no longer U1.2
- new net: NT1.2, U1.2
Changed lines of the file:
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@@
+    (stroke (width 0) (type default))
+  )
+  (wire (pts (xy 44.45 200.66) (xy 49.53 200.66))
     (stroke (width 0) (type default))
   )
@@
     (stroke (width 0) (type default))
   )
+  (wire (pts (xy 33.02 200.66) (xy 39.37 200.66))
+    (stroke (width 0) (type default))
+  )
   (wire (pts (xy 57.15 64.77) (xy 59.69 64.77))
     (stroke (width 0) (type default))
@@
   )
   (wire (pts (xy 45.72 195.58) (xy 49.53 195.58))
-    (stroke (width 0) (type default))
-  )
-  (wire (pts (xy 33.02 200.66) (xy 49.53 200.66))
     (stroke (width 0) (type default))
   )
@@
         )
       )
+    )
+  )
+  (symbol (lib_id "Device:NetTie_2") (at 41.91 200.66 0) (unit 1)
+    (in_bom no) (on_board yes) (dnp no) (fields_autoplaced)
+    (property "Reference" "NT1" (at 41.91 196.85 0)
+      (effects (font (size 1.27 1.27)))
+    )
+    (property "Value" "NetTie_2" (at 41.91 199.39 0)
+      (effects (font (size 1.27 1.27)))
+    )
+    (property "Footprint" "NetTie:NetTie-2_SMD_Pad0.5mm" (at 41.91 200.66 0)
+      (effects (font (size 1.27 1.27)) hide)
+    )
+    (property "Datasheet" "~" (at 41.91 200.66 0)
+      (effects (font (size 1.27 1.27)) hide)
+    )
+    (pin "1")
+    (pin "2")
+    (instances
+      (project "Autogradina"
+        (path "/d51b26fb-d168-4a7a-965a-6a8ab4c74219"
+          (reference "NT1") (unit 1)
+        )
+      )

Commit message: Removed most of traces; Updated schematci
Parts:
- added J10: Conn_01x04_Socket, symbol Connector:Conn_01x04_Socket
Connections:
- net GND: now also J10.2 (Pin_2), J10.4 (Pin_4)
- net Mosfet_Port1: now also U2.17 (GPIO9/TOUCH9/ADC1_CH8/FSPIHD/SUBSPIHD); no longer U2.20 (GPIO12/TOUCH12/ADC2_CH1/FSPICLK/FSPIIO6/SUBSPICLK)
- net Mosfet_Port2: now also U2.18 (GPIO10/TOUCH10/ADC1_CH9/FSPICS0/FSPIIO4/SUBSPICS0); no longer U2.21 (GPIO13/TOUCH13/ADC2_CH2/FSPIQ/FSPIIO7/SUBSPIQ)
- net Mosfet_Port3: now also U2.19 (GPIO11/TOUCH11/ADC2_CH0/FSPID/FSPIIO5/SUBSPID); no longer U2.22 (GPIO14/TOUCH14/ADC2_CH3/FSPIWP/FSPIDQS/SUBSPIWP)
- net Mosfet_Port4: now also U2.20 (GPIO12/TOUCH12/ADC2_CH1/FSPICLK/FSPIIO6/SUBSPICLK); no longer U2.10 (GPIO17/U1TXD/ADC2_CH6)
- net Mosfet_Port5: now also U2.21 (GPIO13/TOUCH13/ADC2_CH2/FSPIQ/FSPIIO7/SUBSPIQ); no longer U2.11 (GPIO18/U1RXD/ADC2_CH7/CLK_OUT3)
- net RELAY1_CONTROL: now also U2.6 (GPIO6/TOUCH6/ADC1_CH5); no longer U2.12 (GPIO8/TOUCH8/ADC1_CH7/SUBSPICS1)
- net RELAY2_CONTROL: now also U2.7 (GPIO7/TOUCH7/ADC1_CH6); no longer U2.17 (GPIO9/TOUCH9/ADC1_CH8/FSPIHD/SUBSPIHD)
- net RELAY3_CONTROL: now also U2.12 (GPIO8/TOUCH8/ADC1_CH7/SUBSPICS1); no longer U2.18 (GPIO10/TOUCH10/ADC1_CH9/FSPICS0/FSPIIO4/SUBSPICS0)
- net General1: now reaches U2.4 (GPIO4/TOUCH4/ADC1_CH3)
- net General1: now also J10.1 (Pin_1)
- net General2: now reaches U2.5 (GPIO5/TOUCH5/ADC1_CH4)
- net General2: now also J10.3 (Pin_3)
Other:
- note added: "Ports used for sensing"
